File: ProPico.kicad_pcb (KiCad board)
At the start: 2 copper layers, 21 x 51 mm, 56 parts, among them J1 USB_C_Receptacle_USB2.0, J2 SWD, J3 LEFT, J4 RIGHT, SW1 BOOTSEL, SW2 RES, U1 FM24CL16B, U2 W25Q16JVUXIQ, U3 AMS1117-3.3, U4 LM4040DBZ-3, U5 RP2040, Y1 ECS-120-12-36-AGN-TR3

Commit message: Updates to get clean BOM output from fabrication toolkit
Parts:
- removed G***: LOGO, LOGO
Connections:
- J4 pad 15: /ADC_VREF -> /ADC_AVDD

Commit message: Updated LCSC references for cheaper assembly
Parts:
- C7: value 10n C0G -> 470n
- R10, R11: value 1k -> 3.3k
- R6: value 470mOhm -> 2.2
Changed lines of the file:
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@@
 			)
 		)
-		(property "LCSC" "C77009"
+		(property "LCSC" "C52923"
 			(at 0 0 0)
 			(layer "F.Fab")
@@
 			)
 		)
-		(property "LCSC" "C57895"
+		(property "LCSC" "C23630"
 			(at 0 0 0)
 			(layer "F.Fab")
@@
 			)
 		)
-		(property "LCSC" "C126499"
+		(property "LCSC" "C1549"
 			(at 0 0 0)
 			(layer "F.Fab")
@@
 			)
 		)
-		(property "LCSC" "C77020"
+		(property "LCSC" "C1525"
 			(at 0 0 0)
 			(layer "F.Fab")
@@
 			)
 		)
-		(property "LCSC" "C25543"
+		(property "LCSC" "C11702"
 			(at 0 0 180)
 			(unlocked yes)
@@
 			)
 		)
-		(property "LCSC" "C105873"
+		(property "LCSC" "C25905"
 			(at 0 0 0)
 			(layer "F.Fab")
@@
 			)
 		)
-		(property "LCSC" "C77020"
+		(property "LCSC" "C1525"
 			(at 0 0 0)
 			(layer "F.Fab")
@@
 			)
 		)
-		(property "LCSC" "C77020"
+		(property "LCSC" "C1525"
 			(at 0 0 0)
 			(layer "F.Fab")
@@
 			)
 		)
-		(property "LCSC" "C126499"
+		(property "LCSC" "C1549"
 			(at 0 0 0)
 			(layer "F.Fab")
@@
 			)
 		)
-		(property "LCSC" "C347222"
+		(property "LCSC" "C6186"
 			(at 0 0 0)
 			(layer "F.Fab")
@@
 			)
 		)
-		(property "LCSC" "C25543"
+		(property "LCSC" "C11702"
 			(at 0 0 0)
 			(layer "F.Fab")
@@
 			)
 		)
-		(property "LCSC" "C77020"
+		(property "LCSC" "C1525"
 			(at 0 0 0)
 			(layer "F.Fab")
@@
 			)
 		)
-		(property "Value" "10n C0G"
+		(property "Value" "470n"
 			(at 0 1.43 0)
 			(layer "F.Fab")
@@
 			)
 		)
-		(property "LCSC" "C76599"
+		(property "LCSC" "C1623"
 			(at 0 0 0)
 			(layer "F.Fab")
@@
 			)
 		)
-		(property "LCSC" "C77020"
+		(property "LCSC" "C1525"
 			(at 0 0 0)
 			(layer "F.Fab")
@@
 			)
 		)
-		(property "LCSC" "C77020"
+		(property "LCSC" "C1525"
 			(at 0 0 0)
 			(layer "F.Fab")
@@
 			)
 		)
-		(property "LCSC" "C552930"
+		(property "LCSC" "C8598"
 			(at 0 0 0)
 			(layer "F.Fab")
@@
 			)
 		)
-		(property "Value" "470mOhm"
+		(property "Value" "2.2"
 			(at 0 1.65 90)
 			(layer "F.Fab")
@@
 			)
 		)
-		(property "LCSC" "C2930220"
+		(property "LCSC" "C17521"
 			(at 0 0 0)
 			(layer "F.Fab")
@@
 			)
 		)
-		(property "LCSC" "C25543"
+		(property "LCSC" "C11702"
 			(at 0 0 0)
 			(layer "F.Fab")
@@
 			)
 		)
-		(property "Value" "1k"
+		(property "Value" "3.3k"
 			(at 0 1.17 0)
 			(layer "F.Fab")
@@
 			)
 		)
-		(property "LCSC" "C25543"
+		(property "LCSC" "C25890"
 			(at 0 0 0)
 			(layer "F.Fab")
@@
 			)
 		)
-		(property "LCSC" "C77020"
+		(property "LCSC" "C1525"
 			(at 0 0 0)
 			(layer "F.Fab")
@@
 			)
 		)
-		(property "Value" "1k"
+		(property "Value" "3.3k"
 			(at 0 1.17 0)
 			(layer "F.Fab")
@@
 			)
 		)
-		(property "LCSC" "C25543"
+		(property "LCSC" "C25890"
 			(at 0 0 0)
 			(layer "F.Fab")
@@
 			)
 		)
-		(property "LCSC" "C105873"
+		(property "LCSC" "C25905"
 			(at 0 0 0)
 			(layer "F.Fab")
@@
 			)
 		)
-		(property "LCSC" "C77020"
+		(property "LCSC" "C1525"
 			(at 0 0 0)
 			(layer "F.Fab")
@@
 			)
 		)
-		(property "LCSC" "C162422"
+		(property "LCSC" "C15850"
 			(at 0 0 0)
 			(layer "F.Fab")
@@
 			)
 		)
-		(property "LCSC" "C77020"
+		(property "LCSC" "C1525"
 			(at 0 0 0)
 			(layer "F.Fab")
@@
 			)
 		)
-		(property "LCSC" "C77009"
+		(property "LCSC" "C52923"
 			(at 0 0 0)
 			(layer "F.Fab")
@@
 			)
 		)
-		(property "LCSC" "C77020"
+		(property "LCSC" "C1525"
 			(at 0 0 0)
 			(layer "F.Fab")
@@
 			)
 		)
-		(property "LCSC" "C434425"
+		(property "LCSC" "C2286"
 			(at 0 0 0)
 			(layer "F.Fab")
@@
 			)
 		)
-		(property "LCSC" "C77020"
+		(property "LCSC" "C1525"
 			(at 0 0 0)
 			(layer "F.Fab")
